Commit message: update urdf

File: urdf/hokuyo_ust.urdf.xacro (robot description, xacro)
@@ -1,5 +1,5 @@
 <?xml version="1.0"?>
 <robot xmlns:xacro="http://ros.org/wiki/xacro">
-  <xacro:macro name="hokuyo_ust_mount" params="prefix parent topic model:=ust-20 *origin">
+  <xacro:macro name="hokuyo_ust_mount" params="prefix parent topic model:=ust-20 min_angle=-2.35619 max_angle=2.35619 visualize:=false *origin">
     <joint name="${prefix}_laser_mount_joint" type="fixed">
       <xacro:insert_block name="origin" />
@@ -24,8 +24,8 @@
     </joint>
     <xacro:if value="${model == 'ust-10'}">
-      <xacro:hokuyo_ust10 frame="${prefix}_laser" topic="${topic}"/>
+      <xacro:hokuyo_ust10 frame="${prefix}_laser" topic="${topic}" min_angle="${min_angle}" max_angle="${max_angle}" visualize="${visualize}" />
     </xacro:if>
     <xacro:if value="${model == 'ust-20'}">
-      <xacro:hokuyo_ust20 frame="${prefix}_laser" topic="${topic}"/>
+      <xacro:hokuyo_ust20 frame="${prefix}_laser" topic="${topic}" min_angle="${min_angle}" max_angle="${max_angle}" visualize="${visualize}" />
     </xacro:if>
     <!-- <gazebo reference="${prefix}_laser_mount">
@@ -34,5 +34,5 @@
   </xacro:macro>
   <!-- Define Hokuyo models -->
-  <xacro:macro name="hokuyo_ust10" params="frame:=laser topic:=scan sample_size:=720 update_rate:=50 min_angle:=-2.35619 max_angle:=2.35619 min_range:=0.1 max_range:=30.0 robot_namespace:=/">
+  <xacro:macro name="hokuyo_ust10" params="frame:=laser topic:=scan sample_size:=720 update_rate:=50 min_angle:=-2.35619 max_angle:=2.35619 min_range:=0.1 max_range:=30.0 visualize:=false robot_namespace:=/">
     <link name="${frame}">
       <inertial>
@@ -44,7 +44,7 @@
       </inertial>
     </link>
-    <xacro:hokuyo_laser_gazebo_v0 frame="${frame}" topic="${topic}" update_rate="50.0" sample_size="${sample_size}" min_angle="${min_angle}" max_angle="${max_angle}" min_range="${min_range}" max_range="${max_range}"/>
+    <xacro:hokuyo_laser_gazebo_v0 frame="${frame}" topic="${topic}" update_rate="50.0" sample_size="${sample_size}" min_angle="${min_angle}" max_angle="${max_angle}" min_range="${min_range}" max_range="${max_range}" visualize="${visualize}" />
   </xacro:macro>
-  <xacro:macro name="hokuyo_ust20" params="frame:=laser topic:=scan sample_size:=720 update_rate:=50 min_angle:=-2.35619 max_angle:=2.35619 min_range:=0.1 max_range:=60.0 robot_namespace:=/">
+  <xacro:macro name="hokuyo_ust20" params="frame:=laser topic:=scan sample_size:=720 update_rate:=50 min_angle:=-2.35619 max_angle:=2.35619 min_range:=0.1 max_range:=60.0 visualize:=false robot_namespace:=/">
     <link name="${frame}">
       <inertial>
@@ -56,13 +56,13 @@
       </inertial>
     </link>
-    <xacro:hokuyo_laser_gazebo_v0 frame="${frame}" topic="${topic}" update_rate="50.0" sample_size="${sample_size}" min_angle="${min_angle}" max_angle="${max_angle}" min_range="${min_range}" max_range="${max_range}"/>
+    <xacro:hokuyo_laser_gazebo_v0 frame="${frame}" topic="${topic}" update_rate="50.0" sample_size="${sample_size}" min_angle="${min_angle}" max_angle="${max_angle}" min_range="${min_range}" max_range="${max_range}" visualize="${visualize}" />
   </xacro:macro>
   <!-- Gazebo simulation -->
-  <xacro:macro name="hokuyo_laser_gazebo_v0" params="frame topic update_rate sample_size min_angle max_angle min_range max_range">
+  <xacro:macro name="hokuyo_laser_gazebo_v0" params="frame topic update_rate sample_size min_angle max_angle min_range max_range visualize">
       <gazebo reference="${frame}">
         <turnGravityOff>true</turnGravityOff>
         <sensor type="ray" name="${frame}">
           <pose>0 0 0 0 0 0</pose>
-          <visualize>false</visualize>
+          <visualize>${visualize}</visualize>
           <update_rate>${update_rate}</update_rate>
           <ray>

Commit message: [UPD] allow update rate to be set up from urdf

File: urdf/hokuyo_ust.urdf.xacro (robot description, xacro)
@@ -34,5 +34,5 @@
   </xacro:macro>
   <!-- Define Hokuyo models -->
-  <xacro:macro name="hokuyo_ust10" params="frame:=laser topic:=scan sample_size:=720 update_rate:=50 min_angle:=-2.35619 max_angle:=2.35619 min_range:=0.1 max_range:=30.0 visualize:=false robot_namespace:=/">
+  <xacro:macro name="hokuyo_ust10" params="frame:=laser topic:=scan sample_size:=720 update_rate:=1 min_angle:=-2.35619 max_angle:=2.35619 min_range:=0.1 max_range:=10.0 visualize:=false robot_namespace:=/">
     <link name="${frame}">
       <inertial>
@@ -44,7 +44,7 @@
       </inertial>
     </link>
-    <xacro:hokuyo_laser_gazebo_v0 frame="${frame}" topic="${topic}" update_rate="50.0" sample_size="${sample_size}" min_angle="${min_angle}" max_angle="${max_angle}" min_range="${min_range}" max_range="${max_range}" visualize="${visualize}" />
+    <xacro:hokuyo_laser_gazebo_v0 frame="${frame}" topic="${topic}" update_rate="${update_rate}" sample_size="${sample_size}" min_angle="${min_angle}" max_angle="${max_angle}" min_range="${min_range}" max_range="${max_range}" visualize="${visualize}" />
   </xacro:macro>
-  <xacro:macro name="hokuyo_ust20" params="frame:=laser topic:=scan sample_size:=720 update_rate:=50 min_angle:=-2.35619 max_angle:=2.35619 min_range:=0.1 max_range:=60.0 visualize:=false robot_namespace:=/">
+  <xacro:macro name="hokuyo_ust20" params="frame:=laser topic:=scan sample_size:=720 update_rate:=1 min_angle:=-2.35619 max_angle:=2.35619 min_range:=0.1 max_range:=20.0 visualize:=false robot_namespace:=/">
     <link name="${frame}">
       <inertial>
@@ -56,5 +56,5 @@
       </inertial>
     </link>
-    <xacro:hokuyo_laser_gazebo_v0 frame="${frame}" topic="${topic}" update_rate="50.0" sample_size="${sample_size}" min_angle="${min_angle}" max_angle="${max_angle}" min_range="${min_range}" max_range="${max_range}" visualize="${visualize}" />
+    <xacro:hokuyo_laser_gazebo_v0 frame="${frame}" topic="${topic}" update_rate="${update_rate}" sample_size="${sample_size}" min_angle="${min_angle}" max_angle="${max_angle}" min_range="${min_range}" max_range="${max_range}" visualize="${visualize}" />
   </xacro:macro>
   <!-- Gazebo simulation -->

Commit message: [UPD] add robot ns

File: urdf/hokuyo_ust.urdf.xacro (robot description, xacro)
@@ -1,5 +1,5 @@
 <?xml version="1.0"?>
 <robot xmlns:xacro="http://ros.org/wiki/xacro">
-  <xacro:macro name="hokuyo_ust_mount" params="prefix parent topic model:=ust-20 min_angle=-2.35619 max_angle=2.35619 visualize:=false *origin">
+  <xacro:macro name="hokuyo_ust_mount" params="prefix parent topic robot_namespace model:=ust-20 min_angle=-2.35619 max_angle=2.35619 visualize:=false *origin">
     <joint name="${prefix}_laser_mount_joint" type="fixed">
       <xacro:insert_block name="origin" />
@@ -24,8 +24,8 @@
     </joint>
     <xacro:if value="${model == 'ust-10'}">
-      <xacro:hokuyo_ust10 frame="${prefix}_laser" topic="${topic}" min_angle="${min_angle}" max_angle="${max_angle}" visualize="${visualize}" />
+      <xacro:hokuyo_ust10 frame="${prefix}_laser" topic="${topic}" robot_namespace="${robot_namespace}" min_angle="${min_angle}" max_angle="${max_angle}" visualize="${visualize}" />
     </xacro:if>
     <xacro:if value="${model == 'ust-20'}">
-      <xacro:hokuyo_ust20 frame="${prefix}_laser" topic="${topic}" min_angle="${min_angle}" max_angle="${max_angle}" visualize="${visualize}" />
+      <xacro:hokuyo_ust20 frame="${prefix}_laser" topic="${topic}" robot_namespace="${robot_namespace}" min_angle="${min_angle}" max_angle="${max_angle}" visualize="${visualize}" />
     </xacro:if>
     <!-- <gazebo reference="${prefix}_laser_mount">
@@ -34,5 +34,5 @@
   </xacro:macro>
   <!-- Define Hokuyo models -->
-  <xacro:macro name="hokuyo_ust10" params="frame:=laser topic:=scan sample_size:=720 update_rate:=1 min_angle:=-2.35619 max_angle:=2.35619 min_range:=0.1 max_range:=10.0 visualize:=false robot_namespace:=/">
+  <xacro:macro name="hokuyo_ust10" params="frame:=laser topic:=scan sample_size:=720 update_rate:=1 min_angle:=-2.35619 max_angle:=2.35619 min_range:=0.1 max_range:=10.0 visualize:=false robot_namespace">
     <link name="${frame}">
       <inertial>
@@ -44,7 +44,7 @@
       </inertial>
     </link>
-    <xacro:hokuyo_laser_gazebo_v0 frame="${frame}" topic="${topic}" update_rate="${update_rate}" sample_size="${sample_size}" min_angle="${min_angle}" max_angle="${max_angle}" min_range="${min_range}" max_range="${max_range}" visualize="${visualize}" />
+    <xacro:hokuyo_laser_gazebo_v0 frame="${frame}" topic="${topic}" update_rate="${update_rate}" sample_size="${sample_size}" min_angle="${min_angle}" max_angle="${max_angle}" min_range="${min_range}" max_range="${max_range}" visualize="${visualize}" robot_namespace="${robot_namespace}" />
   </xacro:macro>
-  <xacro:macro name="hokuyo_ust20" params="frame:=laser topic:=scan sample_size:=720 update_rate:=1 min_angle:=-2.35619 max_angle:=2.35619 min_range:=0.1 max_range:=20.0 visualize:=false robot_namespace:=/">
+  <xacro:macro name="hokuyo_ust20" params="frame:=laser topic:=scan sample_size:=720 update_rate:=1 min_angle:=-2.35619 max_angle:=2.35619 min_range:=0.1 max_range:=20.0 visualize:=false robot_namespace">
     <link name="${frame}">
       <inertial>
@@ -56,8 +56,8 @@
       </inertial>
     </link>
-    <xacro:hokuyo_laser_gazebo_v0 frame="${frame}" topic="${topic}" update_rate="${update_rate}" sample_size="${sample_size}" min_angle="${min_angle}" max_angle="${max_angle}" min_range="${min_range}" max_range="${max_range}" visualize="${visualize}" />
+    <xacro:hokuyo_laser_gazebo_v0 frame="${frame}" topic="${topic}" update_rate="${update_rate}" sample_size="${sample_size}" min_angle="${min_angle}" max_angle="${max_angle}" min_range="${min_range}" max_range="${max_range}" visualize="${visualize}" robot_namespace="${robot_namespace}" />
   </xacro:macro>
   <!-- Gazebo simulation -->
-  <xacro:macro name="hokuyo_laser_gazebo_v0" params="frame topic update_rate sample_size min_angle max_angle min_range max_range visualize">
+  <xacro:macro name="hokuyo_laser_gazebo_v0" params="frame topic update_rate sample_size min_angle max_angle min_range max_range visualize robot_namespace">
       <gazebo reference="${frame}">
         <turnGravityOff>true</turnGravityOff>
@@ -88,6 +88,6 @@
           <plugin name="gazebo_ros_laser" filename="libgazebo_ros_laser.so">
             <topicName>${topic}</topicName>
-            <frameName>${frame}</frameName>
-            <!-- <robotNamespace>${robot_namespace}</robotNamespace> -->
+            <frameName>${robot_namespace}${frame}</frameName>
+            <robotNamespace>/${robot_namespace}</robotNamespace>
           </plugin>
         </sensor>

Commit message: Update urdf/hokuyo_ust.urdf.xacro

File: urdf/hokuyo_ust.urdf.xacro (robot description, xacro)
@@ -1,5 +1,5 @@
 <?xml version="1.0"?>
 <robot xmlns:xacro="http://ros.org/wiki/xacro">
-  <xacro:macro name="hokuyo_ust_mount" params="prefix parent topic robot_namespace model:=ust-20 min_angle=-2.35619 max_angle=2.35619 visualize:=false *origin">
+  <xacro:macro name="hokuyo_ust_mount" params="prefix parent topic robot_namespace:=/ model:=ust-20 min_angle=-2.35619 max_angle=2.35619 visualize:=false *origin">
     <joint name="${prefix}_laser_mount_joint" type="fixed">
       <xacro:insert_block name="origin" />

Commit message: Update urdf/hokuyo_ust.urdf.xacro

File: urdf/hokuyo_ust.urdf.xacro (robot description, xacro)
@@ -34,5 +34,5 @@
   </xacro:macro>
   <!-- Define Hokuyo models -->
-  <xacro:macro name="hokuyo_ust10" params="frame:=laser topic:=scan sample_size:=720 update_rate:=1 min_angle:=-2.35619 max_angle:=2.35619 min_range:=0.1 max_range:=10.0 visualize:=false robot_namespace">
+  <xacro:macro name="hokuyo_ust10" params="frame:=laser topic:=scan sample_size:=720 update_rate:=1 min_angle:=-2.35619 max_angle:=2.35619 min_range:=0.1 max_range:=10.0 visualize:=false robot_namespace:=/">
     <link name="${frame}">
       <inertial>

Commit message: Update urdf/hokuyo_ust.urdf.xacro

File: urdf/hokuyo_ust.urdf.xacro (robot description, xacro)
@@ -46,5 +46,5 @@
     <xacro:hokuyo_laser_gazebo_v0 frame="${frame}" topic="${topic}" update_rate="${update_rate}" sample_size="${sample_size}" min_angle="${min_angle}" max_angle="${max_angle}" min_range="${min_range}" max_range="${max_range}" visualize="${visualize}" robot_namespace="${robot_namespace}" />
   </xacro:macro>
-  <xacro:macro name="hokuyo_ust20" params="frame:=laser topic:=scan sample_size:=720 update_rate:=1 min_angle:=-2.35619 max_angle:=2.35619 min_range:=0.1 max_range:=20.0 visualize:=false robot_namespace">
+  <xacro:macro name="hokuyo_ust20" params="frame:=laser topic:=scan sample_size:=720 update_rate:=1 min_angle:=-2.35619 max_angle:=2.35619 min_range:=0.1 max_range:=20.0 visualize:=false robot_namespace:=/">
     <link name="${frame}">
       <inertial>

Commit message: [FIX] urdf for ros2, disable gazebo (todo)

File: urdf/hokuyo_ust.urdf.xacro (robot description, xacro)
@@ -12,5 +12,5 @@
         <geometry>
           <!-- Origin of this mesh is the base of the bracket. -->
-          <mesh filename="package://urg_node/meshes/hokuyo_ust.stl" />
+          <mesh filename="file://$(find urg_node)/meshes/hokuyo_ust.stl" />
         </geometry>
         <material name="dark_grey" />
@@ -44,5 +44,5 @@
       </inertial>
     </link>
-    <xacro:hokuyo_laser_gazebo_v0 frame="${frame}" topic="${topic}" update_rate="50.0" sample_size="${sample_size}" min_angle="${min_angle}" max_angle="${max_angle}" min_range="${min_range}" max_range="${max_range}"/>
+    <!-- <xacro:hokuyo_laser_gazebo_v0 frame="${frame}" topic="${topic}" update_rate="50.0" sample_size="${sample_size}" min_angle="${min_angle}" max_angle="${max_angle}" min_range="${min_range}" max_range="${max_range}"/> -->
   </xacro:macro>
   <xacro:macro name="hokuyo_ust20" params="frame:=laser topic:=scan sample_size:=720 update_rate:=50 min_angle:=-2.35619 max_angle:=2.35619 min_range:=0.1 max_range:=60.0 robot_namespace:=/">
@@ -56,7 +56,7 @@
       </inertial>
     </link>
-    <xacro:hokuyo_laser_gazebo_v0 frame="${frame}" topic="${topic}" update_rate="50.0" sample_size="${sample_size}" min_angle="${min_angle}" max_angle="${max_angle}" min_range="${min_range}" max_range="${max_range}"/>
+    <!-- <xacro:hokuyo_laser_gazebo_v0 frame="${frame}" topic="${topic}" update_rate="50.0" sample_size="${sample_size}" min_angle="${min_angle}" max_angle="${max_angle}" min_range="${min_range}" max_range="${max_range}"/> -->
   </xacro:macro>
-  <!-- Gazebo simulation -->
+  <!-- TODO - Gazebo simulation -->
   <xacro:macro name="hokuyo_laser_gazebo_v0" params="frame topic update_rate sample_size min_angle max_angle min_range max_range">
       <gazebo reference="${frame}">
@@ -89,5 +89,5 @@
             <topicName>${topic}</topicName>
             <frameName>${frame}</frameName>
-            <!-- <robotNamespace>${robot_namespace}</robotNamespace> -->
+            <robotNamespace>${robot_namespace}</robotNamespace>
           </plugin>
         </sensor>

Commit message: [FEAT] gazebo gpu lidar

File: urdf/hokuyo_ust.urdf.xacro (robot description, xacro)
@@ -1,5 +1,5 @@
 <?xml version="1.0"?>
 <robot xmlns:xacro="http://ros.org/wiki/xacro">
-  <xacro:macro name="hokuyo_ust_mount" params="prefix parent topic model:=ust-20 *origin">
+  <xacro:macro name="hokuyo_ust_mount" params="prefix parent topic model:=ust-20 robot_name:=/  *origin">
     <joint name="${prefix}_laser_mount_joint" type="fixed">
       <xacro:insert_block name="origin" />
@@ -24,8 +24,8 @@
     </joint>
     <xacro:if value="${model == 'ust-10'}">
-      <xacro:hokuyo_ust10 frame="${prefix}_laser" topic="${topic}"/>
+      <xacro:hokuyo_ust10 frame="${prefix}_laser" topic="${topic}" robot_namespace="${robot_name}"/>
     </xacro:if>
     <xacro:if value="${model == 'ust-20'}">
-      <xacro:hokuyo_ust20 frame="${prefix}_laser" topic="${topic}"/>
+      <xacro:hokuyo_ust20 frame="${prefix}_laser" topic="${topic}" robot_namespace="${robot_name}"/>
     </xacro:if>
     <!-- <gazebo reference="${prefix}_laser_mount">
@@ -44,5 +44,5 @@
       </inertial>
     </link>
-    <!-- <xacro:hokuyo_laser_gazebo_v0 frame="${frame}" topic="${topic}" update_rate="50.0" sample_size="${sample_size}" min_angle="${min_angle}" max_angle="${max_angle}" min_range="${min_range}" max_range="${max_range}"/> -->
+    <xacro:hokuyo_laser_gazebo_v0 frame="${frame}" topic="${topic}" update_rate="50.0" sample_size="${sample_size}" min_angle="${min_angle}" max_angle="${max_angle}" min_range="${min_range}" max_range="${max_range}" robot_namespace="${robot_namespace}"/>
   </xacro:macro>
   <xacro:macro name="hokuyo_ust20" params="frame:=laser topic:=scan sample_size:=720 update_rate:=50 min_angle:=-2.35619 max_angle:=2.35619 min_range:=0.1 max_range:=60.0 robot_namespace:=/">
@@ -56,13 +56,13 @@
       </inertial>
     </link>
-    <!-- <xacro:hokuyo_laser_gazebo_v0 frame="${frame}" topic="${topic}" update_rate="50.0" sample_size="${sample_size}" min_angle="${min_angle}" max_angle="${max_angle}" min_range="${min_range}" max_range="${max_range}"/> -->
+    <xacro:hokuyo_laser_gazebo_v0 frame="${frame}" topic="${topic}" update_rate="50.0" sample_size="${sample_size}" min_angle="${min_angle}" max_angle="${max_angle}" min_range="${min_range}" max_range="${max_range}" robot_namespace="${robot_namespace}"/>
   </xacro:macro>
   <!-- TODO - Gazebo simulation -->
-  <xacro:macro name="hokuyo_laser_gazebo_v0" params="frame topic update_rate sample_size min_angle max_angle min_range max_range">
+  <xacro:macro name="hokuyo_laser_gazebo_v0" params="frame topic update_rate sample_size min_angle max_angle min_range max_range robot_namespace:=/">
       <gazebo reference="${frame}">
-        <turnGravityOff>true</turnGravityOff>
-        <sensor type="ray" name="${frame}">
+        <sensor name='${frame}_sensor' type='gpu_lidar'>"
           <pose>0 0 0 0 0 0</pose>
-          <visualize>false</visualize>
+          <gz_frame_id>${robot_name}/${frame}</gz_frame_id>
+          <topic>${robot_name}/${topic}</topic>
           <update_rate>${update_rate}</update_rate>
           <ray>
@@ -74,4 +74,10 @@
                 <max_angle>${max_angle}</max_angle>
               </horizontal>
+              <vertical>
+                <samples>1</samples>
+                <resolution>0.01</resolution>
+                <min_angle>0</min_angle>
+                <max_angle>0</max_angle>
+            </vertical>
             </scan>
             <range>
@@ -80,15 +86,7 @@
               <resolution>0.01</resolution>
             </range>
-            <noise>
-              <type>gaussian</type>
-              <mean>0.0</mean>
-              <stddev>0.001</stddev>
-            </noise>
           </ray>
-          <plugin name="gazebo_ros_laser" filename="libgazebo_ros_laser.so">
-            <topicName>${topic}</topicName>
-            <frameName>${frame}</frameName>
-            <robotNamespace>${robot_namespace}</robotNamespace>
-          </plugin>
+          <always_on>1</always_on>
+          <visualize>true</visualize>
         </sensor>
       </gazebo>
