Commit message: [FEAT] toogle  as param

File: urdf/hokuyo_ust.urdf.xacro (robot description, xacro)
@@ -1,5 +1,5 @@
 <?xml version="1.0"?>
 <robot xmlns:xacro="http://ros.org/wiki/xacro">
-  <xacro:macro name="hokuyo_ust_mount" params="prefix parent topic model:=ust-20 robot_name:=/  *origin">
+  <xacro:macro name="hokuyo_ust_mount" params="prefix parent topic model:=ust-20 robot_name:=/ enable_tf_prefix:=False *origin">
     <joint name="${prefix}_laser_mount_joint" type="fixed">
       <xacro:insert_block name="origin" />
@@ -24,8 +24,8 @@
     </joint>
     <xacro:if value="${model == 'ust-10'}">
-      <xacro:hokuyo_ust10 frame="${prefix}_laser" topic="${topic}" robot_namespace="${robot_name}"/>
+      <xacro:hokuyo_ust10 frame="${prefix}_laser" topic="${topic}" robot_namespace="${robot_name}" enable_tf_prefix="${enable_tf_prefix}"/>
     </xacro:if>
     <xacro:if value="${model == 'ust-20'}">
-      <xacro:hokuyo_ust20 frame="${prefix}_laser" topic="${topic}" robot_namespace="${robot_name}"/>
+      <xacro:hokuyo_ust20 frame="${prefix}_laser" topic="${topic}" robot_namespace="${robot_name}" enable_tf_prefix="${enable_tf_prefix}"/>
     </xacro:if>
     <!-- <gazebo reference="${prefix}_laser_mount">
@@ -34,5 +34,5 @@
   </xacro:macro>
   <!-- Define Hokuyo models -->
-  <xacro:macro name="hokuyo_ust10" params="frame:=laser topic:=scan sample_size:=720 update_rate:=50 min_angle:=-2.35619 max_angle:=2.35619 min_range:=0.1 max_range:=30.0 robot_namespace:=/">
+  <xacro:macro name="hokuyo_ust10" params="frame:=laser topic:=scan sample_size:=720 update_rate:=50 min_angle:=-2.35619 max_angle:=2.35619 min_range:=0.1 max_range:=30.0 robot_namespace:=/ enable_tf_prefix:=False">
     <link name="${frame}">
       <inertial>
@@ -44,7 +44,7 @@
       </inertial>
     </link>
-    <xacro:hokuyo_laser_gazebo_v0 frame="${frame}" topic="${topic}" update_rate="50.0" sample_size="${sample_size}" min_angle="${min_angle}" max_angle="${max_angle}" min_range="${min_range}" max_range="${max_range}" robot_namespace="${robot_namespace}"/>
+    <xacro:hokuyo_laser_gazebo_v0 frame="${frame}" topic="${topic}" update_rate="50.0" sample_size="${sample_size}" min_angle="${min_angle}" max_angle="${max_angle}" min_range="${min_range}" max_range="${max_range}" robot_namespace="${robot_namespace}" enable_tf_prefix="${enable_tf_prefix}"/>
   </xacro:macro>
-  <xacro:macro name="hokuyo_ust20" params="frame:=laser topic:=scan sample_size:=720 update_rate:=50 min_angle:=-2.35619 max_angle:=2.35619 min_range:=0.1 max_range:=60.0 robot_namespace:=/">
+  <xacro:macro name="hokuyo_ust20" params="frame:=laser topic:=scan sample_size:=720 update_rate:=50 min_angle:=-2.35619 max_angle:=2.35619 min_range:=0.1 max_range:=60.0 robot_namespace:=/ enable_tf_prefix:=False">
     <link name="${frame}">
       <inertial>
@@ -56,14 +56,14 @@
       </inertial>
     </link>
-    <xacro:hokuyo_laser_gazebo_v0 frame="${frame}" topic="${topic}" update_rate="10.0" sample_size="${sample_size}" min_angle="${min_angle}" max_angle="${max_angle}" min_range="${min_range}" max_range="${max_range}" robot_namespace="${robot_namespace}"/>
+    <xacro:hokuyo_laser_gazebo_v0 frame="${frame}" topic="${topic}" update_rate="10.0" sample_size="${sample_size}" min_angle="${min_angle}" max_angle="${max_angle}" min_range="${min_range}" max_range="${max_range}" robot_namespace="${robot_namespace}" enable_tf_prefix="${enable_tf_prefix}"/>
   </xacro:macro>
   <!-- TODO - Gazebo simulation -->
-  <xacro:macro name="hokuyo_laser_gazebo_v0" params="frame topic update_rate sample_size min_angle max_angle min_range max_range robot_namespace:=/">
+  <xacro:macro name="hokuyo_laser_gazebo_v0" params="frame topic update_rate sample_size min_angle max_angle min_range max_range robot_namespace:=/ enable_tf_prefix:=False">
       <gazebo reference="${frame}">
         <sensor name='${frame}_sensor' type='gpu_lidar'>"
           <pose>0 0 0 0 0 0</pose>
-          <gz_frame_id>${robot_name}/${frame}</gz_frame_id>
-          <frame_id>${robot_name}/${frame}</frame_id>
-          <topic>${robot_name}/${topic}</topic>
+          <gz_frame_id>${robot_namespace + '/' + frame if enable_tf_prefix else frame}</gz_frame_id>
+          <frame_id>${robot_namespace + '/' + frame if enable_tf_prefix else frame}</frame_id>
+          <topic>${robot_namespace + '/' + topic if enable_tf_prefix else topic}</topic>
           <update_rate>${update_rate}</update_rate>
           <ray>
